File: schematics/Zelle_2_Schaltplan/Zelle_2_Schaltplan.kicad_sch (KiCad schematic)
At the start: 14 parts, among them J1 Raspberry_Pi_4, K1 12V Relais, M1 Pumpe, U1 ESP32-WROOM-32U, U2 DS18B20, U3 DS18B20

Commit message: 2. Schaltplan überarbeitet
Connections:
- net at U1.2 (VDD): now also J1.2 (5V), J1.4 (5V), K1.A2, R3.1, R4.1
- now unconnected: U1.3 (EN)
Other:
- moved on the sheet: K1, M1, R5, R6, RN1, RN2, U1

Commit message: SDO Korrektur (Davids Teil)
Parts:
- added K2: 5V Relais, Relay_THT:Relay_SPDT_Fujitsu_FTR-LYCA005x_FormC_Vertical, symbol Relay:Fujitsu_FTR-LYCA005x
- added M2: Übergangspumpe, symbol Motor:Fan_ALT
- K1: value 12V Relais -> 5V Relais
- M1: value Pumpe -> Filterpumpe
Connections:
- net +12V: now also K2.11
- net GND: now also M2.2 (-)
- net at J1.2 (5V), J1.4 (5V), K1.A2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: now also K2.A2
- new net: K2.14, M2.1 (+)
